Commit message: fix: ibvs scene gripper joint min angle

File: roarm-m2-camera/description_roarm/roarm_description.urdf (robot description, URDF)
Before this commit: robot roarm_description, 6 links, 5 joints
Joints:
- joint link3_to_gripper_link: limit lower=0 upper=1.5 effort=0 velocity=0 -> lower=-1.5 upper=1.5 effort=0 velocity=0
